File: Project3_ArduinoClone.sch (KiCad schematic (older format))
At the start: 13 parts, among them U1 24LC1025, U2 24LC1025, U3 DS1337_v1, U4 ATMEGA328P-AU, Y1 Crystal 32 MHz, Y2 Crystal 16 MHz

Commit message: Add silkscreen text
Parts:
- U3: symbol Pablo_Kicad_library:DS1337_v1 -> Pablo_KiCad:DS1337_v1
Changed lines of the file:
@@
 $EndComp
 $Comp
-L Pablo_Kicad_library:DS1337_v1 U3
+L Pablo_KiCad:DS1337_v1 U3
 U 1 1 5DA3A1C8
 P 2625 1850
