File: Project3_ArduinoClone-roigmonzon-HP-Pavilion-dv7-3.kicad_pcb (KiCad board)
At the start: 2 copper layers, 40.1 x 26.4 mm, 19 parts, among them J1 Serial, J2 Digital pins, J3 ICSP, J4 I2C, U1 24LC1025, U2 24LC1025, U3 DS1337, U4 ATMEGA328P-AU, Y1 Crystal 32MHz, Y2 Crystal 16MHz

Commit message: Final silkscreen, generate gerbers
Parts:
- removed REF**: OSHW-Logo_5.7x6mm_SilkScreen, Symbol:OSHW-Logo_5.7x6mm_SilkScreen
- removed REF**: KiCad-Logo2_5mm_SilkScreen, Symbol:KiCad-Logo2_5mm_SilkScreen
Other:
- board text removed: "Arduino Clone -EEPROM 2MB -RTC -3V or 3V3 powered"
- board text removed: "Designed by Pablo Roig"
